Commit message: Tested different controllers and added python script

File: src/robot_description/urdf/robot.urdf (robot description, URDF)
Before this commit: robot arm, 5 links, 4 joints
Joints:
- joint toe_foot_joint: limit lower=-3.14159265359 upper=3.14159265359 effort=40.0 velocity=1.0 -> lower=-3.14159265359 upper=200.0 effort=40.0 velocity=1000.0
