Commit message: Implemented trajectory control on the new arm with a demo

File: src/robot_description/urdf/tu_nguyen.urdf (robot description, URDF)
Before this commit: robot tu_nguyen, 7 links, 6 joints
Links:
- added link world
Joints:
- added joint world_base_joint: type fixed, parent world, child base_link
- joint joint_1: limit lower=-1.708 upper=1.708 effort=300 velocity=1 -> lower=-3.14 upper=3.14 effort=300 velocity=1
- joint joint_3: limit lower=-1.708 upper=1.708 effort=300 velocity=1 -> lower=-3.14 upper=1.708 effort=300 velocity=1
- joint joint_4: limit lower=-1.708 upper=1.708 effort=300 velocity=1 -> lower=-3.14 upper=3.14 effort=300 velocity=1

Commit message: Separated joints into multiple controllers and added monitor state

File: src/robot_description/urdf/tu_nguyen.urdf (robot description, URDF)
Before this commit: robot tu_nguyen, 8 links, 7 joints
Joints:
- removed joint joint_51
- removed joint joint_52
- added joint joint_5: type revolute, parent link_4, child link_51, origin xyz=0.0015 0.0096756 0.07625 rpy=0 0 0, axis 1 0 0, limit lower=0 upper=0.4 effort=300 velocity=1
- added joint joint_6: type revolute, parent link_4, child link_52, origin xyz=0.0015 0.036676 0.07625 rpy=0 0 0, axis 1 0 0, limit lower=-0.4 upper=0 effort=300 velocity=1
